Commit message: :lipstick: feat: ajustando o urdf para ficar igual ao bill

File: nav_ws/install/bill_description/share/bill_description/urdf/mech/mecanum_wheel.urdf.xacro (robot description, xacro)
@@ -1,10 +1,11 @@
 <?xml version="1.0"?>
 <robot xmlns:xacro="http://www.ros.org/wiki/xacro">
-  <xacro:property name="wheel_radius" value="0.0325" />
-  <xacro:property name="wheel_separation" value="0.169" />
-  <xacro:property name="wheel_width" value="0.03040" />
-  <xacro:property name="wheel_mass" value="9.1" />
-  <xacro:property name="wheel_xoff" value="0.08" />
-  <xacro:property name="wheel_yoff" value="-0.01" />
+  <!-- Novos parâmetros da roda -->
+  <xacro:property name="wheel_radius" value="0.07"/>
+  <xacro:property name="wheel_thickness" value="0.05"/>
+  <xacro:property name="wheel_mass" value="0.2"/>
+  <xacro:property name="wheel_offset_x" value="0.2"/>
+  <xacro:property name="wheel_offset_y" value="${chassis_width/2 + wheel_thickness/2}"/>
+  <xacro:property name="wheel_offset_z" value="0.0"/>
   <xacro:macro name="mecanum_wheel" params="prefix side x_reflect y_reflect">
     <link name="${prefix}${side}_wheel_link">
@@ -12,5 +13,5 @@
         <origin xyz="0 0 0" rpy="${pi/2} 0 0"/>
         <geometry>
-          <mesh filename="file://$(find bill_description)/meshes/robot_3d/visual/${side}_wheel_X3.STL"/>
+          <cylinder radius="${wheel_radius}" length="${wheel_thickness}"/>
         </geometry>
         <material name="dark_gray">
@@ -21,5 +22,5 @@
         <origin xyz="0 0 0" rpy="${pi/2} 0 0"/>
         <geometry>
-          <cylinder radius="${wheel_radius}" length="${wheel_width}"/>
+          <cylinder radius="${wheel_radius}" length="${wheel_thickness}"/>
         </geometry>
       </collision>
@@ -28,7 +29,7 @@
         <mass value="${wheel_mass}"/>
         <inertia
-          ixx="${(wheel_mass/12.0) * (3*wheel_radius*wheel_radius + wheel_width*wheel_width)}" ixy="0" ixz="0"
+          ixx="${(wheel_mass/12.0) * (3*wheel_radius*wheel_radius + wheel_thickness*wheel_thickness)}" ixy="0" ixz="0"
           iyy="${(wheel_mass/2.0) * (wheel_radius*wheel_radius)}" iyz="0"
-          izz="${(wheel_mass/12.0) * (3*wheel_radius*wheel_radius + wheel_width*wheel_width)}"/>
+          izz="${(wheel_mass/12.0) * (3*wheel_radius*wheel_radius + wheel_thickness*wheel_thickness)}"/>
       </inertial>
     </link>
@@ -37,5 +38,5 @@
       <parent link="${prefix}base_link"/>
       <child link="${prefix}${side}_wheel_link"/>
-      <origin xyz="${x_reflect*wheel_xoff} ${y_reflect*(wheel_separation/2+wheel_yoff)} ${-wheel_radius}" rpy="0 0 0"/>
+      <origin xyz="${x_reflect*wheel_offset_x} ${y_reflect*wheel_offset_y} ${wheel_offset_z - wheel_radius}" rpy="0 0 0"/>
     </joint>
     <gazebo reference="${prefix}${side}_wheel_link">
@@ -43,18 +44,18 @@
         <friction>
           <ode>
-              <mu>1.0</mu>
-              <mu2>0.0</mu2>
+            <mu>1.0</mu>
+            <mu2>0.0</mu2>
           </ode>
         </friction>
       </surface>
       <visual>
-          <material>
-              <ambient>0.2 0.2 0.2 1.0</ambient>
-              <diffuse>0.2 0.2 0.2 1.0</diffuse>
-              <specular>0.2 0.2 0.2 1.0</specular>
-              <emissive>0.0 0.0 0.0 0.0</emissive>
-          </material>
+        <material>
+          <ambient>0.2 0.2 0.2 1.0</ambient>
+          <diffuse>0.2 0.2 0.2 1.0</diffuse>
+          <specular>0.2 0.2 0.2 1.0</specular>
+          <emissive>0.0 0.0 0.0 0.0</emissive>
+        </material>
       </visual>
-  </gazebo>
+    </gazebo>
   </xacro:macro>
 </robot>

File: nav_ws/install/bill_description/share/bill_description/urdf/mech/robot_3d_base.urdf.xacro (robot description, xacro)
@@ -1,56 +1,61 @@
 <?xml version="1.0"?>
 <robot xmlns:xacro="http://www.ros.org/wiki/xacro">
-<xacro:property name="total_width" value="0.19940" />
-<xacro:property name="wheel_width" value="0.0304" />
-<xacro:property name="wheel_radius" value="0.0325" />
-<xacro:property name="total_height" value="0.26225" />
-<xacro:property name="base_length" value="0.300" />
-<xacro:property name="centered_length" value="0.238" />
-<xacro:property name="base_x_offset" value="${(centered_length - base_length) / 2}" />
-<xacro:property name="base_size_x" value="${base_length}" />
-<xacro:property name="base_size_y" value="${total_width - (2 * wheel_width)}" />
-<xacro:property name="base_size_z" value="${total_height - (2 * wheel_radius)}" />
-<xacro:property name="base_mass" value="4.6" />
-<xacro:macro name="robot_3d_base" params="prefix">
-  <link name="${prefix}base_footprint"/>
-  <link name="${prefix}base_link">
-    <visual>
+  <!-- Novos parâmetros do chassi e rodas -->
+  <xacro:property name="chassis_length" value="0.5"/>
+  <xacro:property name="chassis_width" value="0.3"/>
+  <xacro:property name="chassis_height" value="1.17"/>
+  <xacro:property name="chassis_mass" value="22.2"/>
+  <xacro:property name="wheel_radius" value="0.07"/>
+  <xacro:property name="wheel_thickness" value="0.05"/>
+  <xacro:property name="wheel_mass" value="0.2"/>
+  <xacro:property name="wheel_offset_x" value="0.2"/>
+  <xacro:property name="wheel_offset_y" value="${chassis_width/2 + wheel_thickness/2}"/>
+  <xacro:property name="wheel_offset_z" value="0.0"/>
+  <!-- Macro do corpo do robô -->
+  <xacro:macro name="robot_3d_base" params="prefix">
+    <link name="${prefix}base_footprint"/>
+    <link name="${prefix}base_link">
+      <visual>
         <geometry>
-            <mesh filename="file://$(find bill_description)/meshes/robot_3d/visual/base_link_X3.STL"/>
+          <box size="${chassis_length} ${chassis_width} ${chassis_height}"/>
         </geometry>
         <material name="white">
           <color rgba="1 1 1 1"/>
         </material>
-        <origin xyz="0 0 0" rpy="0 0 0"/>
-    </visual>
-    <collision>
+        <!-- Centro do chassi fica acima das rodas -->
+        <origin xyz="0 0 ${chassis_height/2 + wheel_radius}" rpy="0 0 0"/>
+      </visual>
+      <collision>
         <geometry>
-            <box size="${base_size_x} ${base_size_y} ${base_size_z}"/>
+          <box size="${chassis_length} ${chassis_width} ${chassis_height}"/>
         </geometry>
-        <origin xyz="${base_x_offset} 0 ${base_size_z/2 + wheel_radius/4}" rpy="0 0 0"/>
-    </collision>
-    <inertial>
-        <origin xyz="${base_x_offset} 0 ${base_size_z/2 + wheel_radius/4}" rpy="0 0 0"/>
-        <mass value="${base_mass}"/>
+        <origin xyz="0 0 ${chassis_height/2 + wheel_radius}" rpy="0 0 0"/>
+      </collision>
+      <inertial>
+        <origin xyz="0 0 ${chassis_height/2 + wheel_radius}" rpy="0 0 0"/>
+        <mass value="${chassis_mass}"/>
         <inertia
-            ixx="${(1/12) * base_mass * ((base_size_y * base_size_y) + (base_size_z * base_size_z))}" ixy="0.0" ixz="0.0"
-            iyy="${(1/12) * base_mass * ((base_size_x * base_size_x) + (base_size_z * base_size_z))}" iyz="0.0"
-            izz="${(1/12) * base_mass * ((base_size_x * base_size_x) + (base_size_y * base_size_y))}"/>
-    </inertial>
-  </link>
-  <gazebo reference="${prefix}base_link">
-    <visual>
+          ixx="${(1/12.0) * chassis_mass * (chassis_width * chassis_width + chassis_height * chassis_height)}"
+          ixy="0.0"
+          ixz="0.0"
+          iyy="${(1/12.0) * chassis_mass * (chassis_length * chassis_length + chassis_height * chassis_height)}"
+          iyz="0.0"
+          izz="${(1/12.0) * chassis_mass * (chassis_length * chassis_length + chassis_width * chassis_width)}"/>
+      </inertial>
+    </link>
+    <gazebo reference="${prefix}base_link">
+      <visual>
         <material>
-            <ambient>0 0.7 0 1</ambient>
-            <diffuse>0 0.7 0 1</diffuse>
-            <specular>0 0.7 0 1</specular>
+          <ambient>0 0.7 0 1</ambient>
+          <diffuse>0 0.7 0 1</diffuse>
+          <specular>0 0.7 0 1</specular>
         </material>
-    </visual>
-  </gazebo>
-  <joint name="${prefix}base_joint" type="fixed">
-    <parent link="${prefix}base_footprint"/>
-    <child link="${prefix}base_link"/>
-    <origin xyz="0 0 ${wheel_radius}" rpy="0 0 0"/>
-  </joint>
-</xacro:macro>
+      </visual>
+    </gazebo>
+    <joint name="${prefix}base_joint" type="fixed">
+      <parent link="${prefix}base_footprint"/>
+      <child link="${prefix}base_link"/>
+      <origin xyz="0 0 0" rpy="0 0 0"/>
+    </joint>
+  </xacro:macro>
 </robot>

File: nav_ws/install/bill_description/share/bill_description/urdf/robots/robot_3d.urdf.xacro (robot description, xacro)
@@ -33,8 +33,6 @@
       parent="base_link"
       frame_id="laser_frame"
-      xyz_offset="0 0 0.0825"
+      xyz_offset="0.3 0 0.3"
       rpy_offset="0 0 3.14"
-      mesh_xyz_offset="0 0 0"
-      mesh_rpy_offset="${-M_PI/2} 0 0"
       topic_name="scan"/>
     <!--

File: nav_ws/install/bill_description/share/bill_description/urdf/sensors/lidar.urdf.xacro (robot description, xacro)
@@ -6,16 +6,12 @@
     parent:='base_link'
     frame_id:='laser_frame'
-    mesh_file:='file://$(find bill_description)/meshes/rplidar/rplidar_s2.stl'
     xyz_offset:='0 0 0.0825'
     rpy_offset:='0 0 0'
-    mesh_xyz_offset:='0 0 0'
-    mesh_rpy_offset:='${-M_PI/2} 0 0'
-    mesh_scale:='0.001 0.001 0.001'
+    lidar_width:=0.077
+    lidar_height:=0.0398
     collision_xyz_offset:='0 0 0'
     collision_rpy_offset:='0 0 0'
     inertial_xyz_offset:='0 0 0'
     inertial_rpy_offset:='0 0 0'
-    lidar_width:=0.077
-    lidar_height:=0.0398
     mass:=0.185
     material_name:='rplidar_black'
@@ -40,7 +36,7 @@
     <link name="${prefix}${frame_id}">
       <visual>
-        <origin xyz="${mesh_xyz_offset}" rpy="${mesh_rpy_offset}"/>
+        <origin xyz="0 0 0" rpy="0 0 0"/>
         <geometry>
-          <mesh filename="${mesh_file}" scale="${mesh_scale}"/>
+          <cylinder radius="${radius}" length="${lidar_height}"/>
         </geometry>
         <material name="${material_name}">
