Commit message: :bricks: feat:adicionando simulação com o gazebo

File: nav_ws/src/bill_description/urdf/robots/robot_3d.urdf.xacro (robot description, xacro)
@@ -1,4 +1,4 @@
 <?xml version="1.0"?>
-<robot xmlns:xacro="http://www.ros.org/wiki/xacro" name="robot_3d">
+<robot xmlns:xacro="http://www.ros.org/wiki/xacro" xmlns:gz="https://gazebosim.org/schemas" name="robot_3d">
     <xacro:property name="M_PI" value="3.1415926535897931" />
     <xacro:arg name="robot_name" default="robot_3d"/>
@@ -8,4 +8,5 @@
     <xacro:include filename="$(find bill_description)/urdf/mech/mecanum_wheel.urdf.xacro"/>
     <xacro:include filename="$(find bill_description)/urdf/sensors/lidar.urdf.xacro"/>
+    <xacro:include filename="$(find bill_description)/urdf/control/bill.gazebo"/>
     <xacro:robot_3d_base prefix="$(arg prefix)"/>
     <xacro:mecanum_wheel
@@ -36,15 +37,60 @@
       rpy_offset="0 0 3.14"
       topic_name="scan"/>
-    <!--
-    <xacro:include filename="$(find bill_description)/urdf/control/velocity_control_plugin.urdf.xacro" />
-    <xacro:load_velocity_control_plugin use_gazebo="$(arg use_gazebo)"/>
-    <xacro:include filename="$(find bill_description)/urdf/control/gazebo_sim_ros2_control.urdf.xacro" />
-    <xacro:load_gazebo_sim_ros2_control_plugin
-      robot_name="$(arg robot_name)"
-      use_gazebo="$(arg use_gazebo)"/>
-    <xacro:include filename="$(find bill_description)/urdf/control/robot_3d_ros2_control.urdf.xacro" />
-    <xacro:bill_ros2_control
-      prefix="$(arg prefix)"
-      use_gazebo="$(arg use_gazebo)"/>
-    -->
+    <gazebo reference='front_left_wheel_link'>
+      <collision>
+        <surface>
+          <friction>
+            <ode>
+              <mu>1.5</mu>
+              <mu2>0.0</mu2>
+              <fdir1 gz:expressed_in="base_footprint">1 -1 0</fdir1>
+            </ode>
+          </friction>
+        </surface>
+      </collision>
+    </gazebo>
+    <gazebo reference='back_left_wheel_link'>
+      <collision>
+        <surface>
+          <friction>
+            <ode>
+              <mu>1.5</mu>
+              <mu2>0.0</mu2>
+              <fdir1 gz:expressed_in="base_footprint">1 1 0</fdir1>
+            </ode>
+          </friction>
+        </surface>
+      </collision>
+    </gazebo>
+    <gazebo reference='front_right_wheel_link'>
+      <collision>
+        <surface>
+          <friction>
+            <ode>
+              <mu>1.5</mu>
+              <mu2>0.0</mu2>
+              <fdir1 gz:expressed_in="base_footprint">1 1 0</fdir1>
+            </ode>
+          </friction>
+        </surface>
+      </collision>
+    </gazebo>
+    <gazebo reference='back_right_wheel_link'>
+      <collision>
+        <surface>
+          <friction>
+            <ode>
+              <mu>1.5</mu>
+              <mu2>0.0</mu2>
+              <fdir1 gz:expressed_in="base_footprint">1 -1 0</fdir1>
+            </ode>
+          </friction>
+        </surface>
+      </collision>
+    </gazebo>
+    <gazebo reference="base_link">
+      <mu1>0.000002</mu1>
+      <mu2>0.000002</mu2>
+      <!-- <material>Gazebo/Red</material> -->
+    </gazebo>
 </robot>
